File: hardware/ensemble.kicad_sch (KiCad schematic)
At the start: 22 parts, among them J1 E1, SW1 4PDT Toggle, SW2 SPDT Toggle, SW3 SPST Toggle, T1 42TM_XX, U1 LM741

Commit message: slight routing and layout changes
Parts:
- SW3: value SPST Toggle -> SPST Toggle (or half an SPDT)
Connections:
- net POST_BALANCE: now reaches D3.2 (A), D5.1 (K), RV2.2, RV3.3
- net 741_Out: now reaches C3.1, R3.2, U1.6
- net 741_Inv: now reaches C1.2, R1.1, R2.2, RV1.1, U1.2 (-)
Other:
- note added: "Choose transformer based on ratio of Primary to Secondary turns. Higher ratio == louder/stronger octave effect, and more clipping. My choice: 42TM011-RC"
Changed lines of the file:
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@@
     (title "Ensemble fuzz effect")
     (date "2023-03-19")
-    (rev "v0.02")
+    (rev "v0.021")
     (comment 1 "github.com/whbeers/ensemble")
   )
@@
     (stroke (width 0) (type default))
   )
+  (wire (pts (xy 156.21 27.94) (xy 172.72 27.94))
+    (stroke (width 0) (type default))
+  )
+  (wire (pts (xy 66.675 118.745) (xy 79.375 118.745))
+    (stroke (width 0) (type default))
+  )
+  (wire (pts (xy 25.4 41.275) (xy 15.24 41.275))
+    (stroke (width 0) (type default))
+  )
+  (wire (pts (xy 133.985 24.13) (xy 133.985 22.225))
+    (stroke (width 0) (type default))
+  )
+  (wire (pts (xy 175.26 80.645) (xy 179.07 80.645))
+    (stroke (width 0) (type default))
+  )
+  (wire (pts (xy 48.895 123.825) (xy 50.8 123.825))
+    (stroke (width 0) (type default))
+  )
+  (wire (pts (xy 53.34 41.275) (xy 57.15 41.275))
+    (stroke (width 0) (type default))
+  )
+  (wire (pts (xy 25.4 50.8) (xy 31.75 50.8))
+    (stroke (width 0) (type default))
+  )
+  (wire (pts (xy 14.605 78.105) (xy 24.765 78.105))
+    (stroke (width 0) (type default))
+  )
+  (wire (pts (xy 130.175 81.915) (xy 130.175 83.185))
+    (stroke (width 0) (type default))
+  )
+  (wire (pts (xy 53.34 26.035) (xy 53.34 41.275))
+    (stroke (width 0) (type default))
+  )
+  (wire (pts (xy 57.15 22.225) (xy 62.865 22.225))
+    (stroke (width 0) (type default))
+  )
+  (wire (pts (xy 89.535 123.825) (xy 89.535 128.905))
+    (stroke (width 0) (type default))
+  )
+  (wire (pts (xy 86.36 88.265) (xy 86.36 88.9))
+    (stroke (width 0) (type default))
+  )
+  (wire (pts (xy 151.13 27.94) (xy 156.21 27.94))
+    (stroke (width 0) (type default))
+  )
+  (wire (pts (xy 105.41 90.805) (xy 98.425 90.805))
+    (stroke (width 0) (type default))
+  )
+  (wire (pts (xy 72.39 38.735) (xy 76.2 38.735))
+    (stroke (width 0) (type default))
+  )
+  (wire (pts (xy 120.015 88.265) (xy 130.175 88.265))
+    (stroke (width 0) (type default))
+  )
+  (wire (pts (xy 130.175 88.265) (xy 139.065 88.265))
+    (stroke (width 0) (type default))
+  )
+  (wire (pts (xy 118.745 33.655) (xy 133.985 33.655))
+    (stroke (width 0) (type default))
+  )
+  (wire (pts (xy 34.925 80.645) (xy 46.99 80.645))
+    (stroke (width 0) (type default))
+  )
+  (wire (pts (xy 39.37 50.8) (xy 45.72 50.8))
+    (stroke (width 0) (type default))
+  )
+  (wire (pts (xy 45.72 50.8) (xy 45.72 41.275))
+    (stroke (width 0) (type default))
+  )
+  (wire (pts (xy 76.2 38.735) (xy 76.2 22.225))
+    (stroke (width 0) (type default))
+  )
   (wire (pts (xy 43.815 41.275) (xy 45.72 41.275))
     (stroke (width 0) (type default))
   )
-  (wire (pts (xy 156.21 27.94) (xy 172.72 27.94))
-    (stroke (width 0) (type default))
-  )
-  (wire (pts (xy 66.675 118.745) (xy 79.375 118.745))
-    (stroke (width 0) (type default))
-  )
-  (wire (pts (xy 25.4 41.275) (xy 15.24 41.275))
-    (stroke (width 0) (type default))
-  )
-  (wire (pts (xy 133.985 24.13) (xy 133.985 22.225))
-    (stroke (width 0) (type default))
-  )
-  (wire (pts (xy 175.26 80.645) (xy 179.07 80.645))
-    (stroke (width 0) (type default))
-  )
-  (wire (pts (xy 48.895 123.825) (xy 50.8 123.825))
-    (stroke (width 0) (type default))
-  )
-  (wire (pts (xy 53.34 41.275) (xy 57.15 41.275))
-    (stroke (width 0) (type default))
-  )
-  (wire (pts (xy 25.4 50.8) (xy 31.75 50.8))
-    (stroke (width 0) (type default))
-  )
-  (wire (pts (xy 14.605 78.105) (xy 24.765 78.105))
-    (stroke (width 0) (type default))
-  )
-  (wire (pts (xy 130.175 81.915) (xy 130.175 83.185))
-    (stroke (width 0) (type default))
-  )
-  (wire (pts (xy 53.34 26.035) (xy 53.34 41.275))
-    (stroke (width 0) (type default))
-  )
-  (wire (pts (xy 57.15 22.225) (xy 62.865 22.225))
-    (stroke (width 0) (type default))
-  )
-  (wire (pts (xy 89.535 123.825) (xy 89.535 128.905))
-    (stroke (width 0) (type default))
-  )
-  (wire (pts (xy 86.36 88.265) (xy 86.36 88.9))
-    (stroke (width 0) (type default))
-  )
-  (wire (pts (xy 151.13 27.94) (xy 156.21 27.94))
-    (stroke (width 0) (type default))
-  )
-  (wire (pts (xy 105.41 90.805) (xy 98.425 90.805))
-    (stroke (width 0) (type default))
-  )
-  (wire (pts (xy 72.39 38.735) (xy 76.2 38.735))
-    (stroke (width 0) (type default))
-  )
-  (wire (pts (xy 120.015 88.265) (xy 130.175 88.265))
-    (stroke (width 0) (type default))
-  )
-  (wire (pts (xy 130.175 88.265) (xy 139.065 88.265))
-    (stroke (width 0) (type default))
-  )
-  (wire (pts (xy 118.745 33.655) (xy 133.985 33.655))
-    (stroke (width 0) (type default))
-  )
-  (wire (pts (xy 34.925 80.645) (xy 46.99 80.645))
-    (stroke (width 0) (type default))
-  )
-  (wire (pts (xy 39.37 50.8) (xy 45.72 50.8))
-    (stroke (width 0) (type default))
-  )
-  (wire (pts (xy 45.72 50.8) (xy 45.72 41.275))
-    (stroke (width 0) (type default))
-  )
-  (wire (pts (xy 76.2 38.735) (xy 76.2 22.225))
-    (stroke (width 0) (type default))
-  )
   (wire (pts (xy 176.53 34.925) (xy 191.135 34.925))
     (stroke (width 0) (type default))
@@
     (stroke (width 0) (type default))
   )
-  (wire (pts (xy 97.79 38.735) (xy 95.885 38.735))
-    (stroke (width 0) (type default))
-  )
   (wire (pts (xy 153.67 45.085) (xy 156.21 45.085))
     (stroke (width 0) (type default))
@@
     (stroke (width 0) (type default))
   )
+  (wire (pts (xy 95.885 38.735) (xy 107.95 38.735))
+    (stroke (width 0) (type default))
+  )
   (wire (pts (xy 49.53 50.8) (xy 49.53 52.705))
     (stroke (width 0) (type default))
@@
   )
   (wire (pts (xy 133.985 31.75) (xy 133.985 33.655))
-    (stroke (width 0) (type default))
-  )
-  (wire (pts (xy 50.8 123.825) (xy 50.8 124.46))
     (stroke (width 0) (type default))
   )
@@
     (effects (font (size 0.8 0.8)) (justify left bottom))
   )
-  (text "See \"Transformer Switching\"" (at 28.575 133.35 0)
+  (text "Choose transformer based on ratio of Primary to Secondary turns.\nHigher ratio == louder/stronger octave effect, and more clipping.\n\nMy choice: 42TM011-RC "
+    (at 23.495 114.935 0)
+    (effects (font (size 1 1)) (justify left bottom))
+  )
+  (text "See \"Transformer Switching\"" (at 29.21 132.715 0)
     (effects (font (size 1 1)) (justify left bottom))
   )
@@
     (effects (font (size 1.27 1.27)) (justify left bottom))
   )
-  (text "R3 sets minimum gain" (at 60.96 17.78 0)
+  (text "R3 sets minimum gain" (at 60.325 18.415 0)
     (effects (font (size 0.8 0.8)) (justify left bottom))
   )
@@
     (effects (font (size 1.27 1.27)) (justify left bottom))
   )
+  (label "741_Out" (at 72.39 38.735 0) (fields_autoplaced)
+    (effects (font (size 1.27 1.27)) (justify left bottom))
+  )
   (label "XFM_P3" (at 44.45 92.075 180) (fields_autoplaced)
     (effects (font (size 1.27 1.27)) (justify right bottom))
@@
     (effects (font (size 1.27 1.27)) (justify left bottom))
   )
+  (label "741_Inv" (at 44.45 41.275 0) (fields_autoplaced)
+    (effects (font (size 1.27 1.27)) (justify left bottom))
+  )
   (label "RECT_TOP" (at 70.485 78.105 180) (fields_autoplaced)
     (effects (font (size 1.27 1.27)) (justify right bottom))
@@
     (effects (font (size 1.27 1.27)) (justify right bottom))
   )
+  (label "POST_BALANCE" (at 161.29 27.94 0) (fields_autoplaced)
+    (effects (font (size 1.27 1.27)) (justify left bottom))
+  )
   (label "GND" (at 175.26 85.725 180) (fields_autoplaced)
     (effects (font (size 1.27 1.27)) (justify right bottom))
@@
     (effects (font (size 1.27 1.27)) (justify right bottom))
   )
-  (label "DRIVE_OUT" (at 97.79 38.735 0) (fields_autoplaced)
-    (effects (font (size 1.27 1.27)) (justify left bottom))
-  )
-  (symbol (lib_id "power:GND") (at 50.8 124.46 0) (unit 1)
+  (label "DRIVE_OUT" (at 107.95 38.735 180) (fields_autoplaced)
+    (effects (font (size 1.27 1.27)) (justify right bottom))
+  )
+  (symbol (lib_id "power:GND") (at 50.8 123.825 0) (unit 1)
     (in_bom yes) (on_board yes) (dnp no) (fields_autoplaced)
-    (property "Reference" "#PWR01" (at 50.8 130.81 0)
-      (effects (font (size 1.27 1.27)) hide)
-    )
-    (property "Value" "GND" (at 50.8 129.54 0)
-      (effects (font (size 1.27 1.27)) hide)
-    )
-    (property "Footprint" "" (at 50.8 124.46 0)
-      (effects (font (size 1.27 1.27)) hide)
-    )
-    (property "Datasheet" "" (at 50.8 124.46 0)
+    (property "Reference" "#PWR01" (at 50.8 130.175 0)
+      (effects (font (size 1.27 1.27)) hide)
+    )
+    (property "Value" "GND" (at 50.8 128.905 0)
+      (effects (font (size 1.27 1.27)) hide)
+    )
+    (property "Footprint" "" (at 50.8 123.825 0)
+      (effects (font (size 1.27 1.27)) hide)
+    )
+    (property "Datasheet" "" (at 50.8 123.825 0)
       (effects (font (size 1.27 1.27)) hide)
     )
@@
       (effects (font (size 1.27 1.27)) hide)
     )
-    (property "Datasheet" "" (at 38.735 131.445 0)
+    (property "Datasheet" "https://www.mouser.com/datasheet/2/449/XC-600134-1212477.pdf" (at 38.735 131.445 0)
       (effects (font (size 1.27 1.27)) hide)
     )
@@
   )
   (symbol (lib_name "SW_4PDT_2") (lib_id "ensemble:SW_4PDT") (at 53.34 75.565 180) (unit 2)
-    (in_bom yes) (on_board yes) (dnp no) (fields_autoplaced)
-    (property "Reference" "SW1" (at 52.07 74.295 0)
+    (in_bom yes) (on_board yes) (dnp no)
+    (property "Reference" "SW1" (at 52.07 73.66 0)
       (effects (font (size 1.27 1.27)))
     )
@@
   )
   (symbol (lib_name "SW_4PDT_3") (lib_id "ensemble:SW_4PDT") (at 28.575 92.075 0) (unit 3)
-    (in_bom yes) (on_board yes) (dnp no) (fields_autoplaced)
-    (property "Reference" "SW1" (at 29.845 85.725 0)
+    (in_bom yes) (on_board yes) (dnp no)
+    (property "Reference" "SW1" (at 29.845 85.09 0)
       (effects (font (size 1.27 1.27)))
     )
@@
       (effects (font (size 1.27 1.27)) (justify right))
     )
-    (property "Value" "SPST Toggle" (at 154.94 52.07 90)
-      (effects (font (size 1.27 1.27)) (justify right))
-    )
+    (property "Value" "SPST Toggle (or half an SPDT)" (at 154.94 52.07 90)
+      (effects (font (size 1.27 1.27)) (justify right))
+    )
