File: hardware/ensemble.kicad_pcb (KiCad board)
At the start: 2 copper layers, 50 x 55 mm, 22 parts, among them J1 E1, SW1 4PDT Toggle, SW2 SPDT Toggle, SW3 SPST Toggle, T1 42TM_XX, U1 LM741

Commit message: getting closer to happy with the layout
Routing:
- net /XFM_S3: track 48.0 -> 42.4 mm
- net /XFM_P3: track 44.4 -> 41.8 mm
- net /XFM_P1: track 42.0 -> 40.3 mm
- net /XFM_S1: track 27.5 -> 26.6 mm
Changed lines of the file:
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@@
   (segment (start 38.4 37.4) (end 43 42) (width 0.25) (layer "F.Cu") (net 16))
   (segment (start 61.4 44.9) (end 45.9 44.9) (width 0.25) (layer "F.Cu") (net 16))
-  (segment (start 64.4 57.1) (end 63.2 55.9) (width 0.25) (layer "F.Cu") (net 21))
-  (segment (start 69.5 57.1) (end 64.4 57.1) (width 0.25) (layer "F.Cu") (net 21))
-  (segment (start 70.4875 56.1125) (end 69.85 56.75) (width 0.25) (layer "F.Cu") (net 21))
-  (segment (start 55.7 50.3) (end 54.55 51.45) (width 0.25) (layer "F.Cu") (net 21))
+  (segment (start 64.4 57.1) (end 69.5 57.1) (width 0.25) (layer "F.Cu") (net 21))
+  (segment (start 54.55 51.45) (end 56.268333 49.731667) (width 0.25) (layer "F.Cu") (net 21))
   (segment (start 62.5 51.2) (end 61.3 50) (width 0.25) (layer "F.Cu") (net 21))
-  (segment (start 63.2 51.9) (end 62.5 51.2) (width 0.25) (layer "F.Cu") (net 21))
-  (segment (start 56.268333 49.731667) (end 55.7 50.3) (width 0.25) (layer "F.Cu") (net 21))
-  (segment (start 69.85 56.75) (end 69.5 57.1) (width 0.25) (layer "F.Cu") (net 21))
+  (segment (start 69.5 57.1) (end 70.4875 56.1125) (width 0.25) (layer "F.Cu") (net 21))
   (segment (start 61.031667 49.731667) (end 62.5 51.2) (width 0.25) (layer "F.Cu") (net 21))
+  (segment (start 62.5 51.2) (end 63.2 51.9) (width 0.25) (layer "F.Cu") (net 21))
+  (segment (start 63.2 51.9) (end 63.2 55.9) (width 0.25) (layer "F.Cu") (net 21))
   (segment (start 54.55 51.45) (end 54.55 53.926) (width 0.25) (layer "F.Cu") (net 21))
-  (segment (start 63.2 55.9) (end 63.2 51.9) (width 0.25) (layer "F.Cu") (net 21))
-  (segment (start 70.5 56.1) (end 69.85 56.75) (width 0.25) (layer "F.Cu") (net 21))
+  (segment (start 63.2 55.9) (end 64.4 57.1) (width 0.25) (layer "F.Cu") (net 21))
   (segment (start 60.9625 49.731667) (end 56.268333 49.731667) (width 0.25) (layer "F.Cu") (net 21))
-  (segment (start 53.8 55.6) (end 52.126 53.926) (width 0.25) (layer "F.Cu") (net 22))
-  (segment (start 52.126 53.926) (end 41.85 53.926) (width 0.25) (layer "F.Cu") (net 22))
-  (segment (start 59.2 55.6) (end 53.8 55.6) (width 0.25) (layer "F.Cu") (net 22))
-  (segment (start 59.931667 54.868333) (end 59.5 55.3) (width 0.25) (layer "F.Cu") (net 22))
-  (segment (start 60.2 54.6) (end 59.5 55.3) (width 0.25) (layer "F.Cu") (net 22))
-  (segment (start 60.9625 54.868333) (end 59.931667 54.868333) (width 0.25) (layer "F.Cu") (net 22))
-  (segment (start 59.5 55.3) (end 59.2 55.6) (width 0.25) (layer "F.Cu") (net 22))
-  (segment (start 60.8 46.5) (end 68.9 46.5) (width 0.25) (layer "B.Cu") (net 22))
-  (segment (start 59 54.1) (end 59 48.3) (width 0.25) (layer "B.Cu") (net 22))
-  (segment (start 60.9625 54.6) (end 59.5 54.6) (width 0.25) (layer "B.Cu") (net 22))
+  (segment (start 52.126 53.926) (end 53.8 55.6) (width 0.25) (layer "F.Cu") (net 22))
+  (segment (start 41.85 53.926) (end 52.126 53.926) (width 0.25) (layer "F.Cu") (net 22))
+  (segment (start 59.2 55.6) (end 60.2 54.6) (width 0.25) (layer "F.Cu") (net 22))
+  (segment (start 53.8 55.6) (end 59.2 55.6) (width 0.25) (layer "F.Cu") (net 22))
+  (segment (start 68.9 46.5) (end 60.8 46.5) (width 0.25) (layer "B.Cu") (net 22))
+  (segment (start 59.5 54.6) (end 60.9625 54.6) (width 0.25) (layer "B.Cu") (net 22))
+  (segment (start 70.4875 48.0875) (end 68.9 46.5) (width 0.25) (layer "B.Cu") (net 22))
+  (segment (start 60.8 46.5) (end 59 48.3) (width 0.25) (layer "B.Cu") (net 22))
   (segment (start 59 54.1) (end 59.5 54.6) (width 0.25) (layer "B.Cu") (net 22))
-  (segment (start 59 48.3) (end 60.8 46.5) (width 0.25) (layer "B.Cu") (net 22))
-  (segment (start 68.9 46.5) (end 70.4875 48.0875) (width 0.25) (layer "B.Cu") (net 22))
-  (segment (start 59.675 59.875) (end 58.512 61.038) (width 0.25) (layer "F.Cu") (net 23))
-  (segment (start 60.9625 59.468333) (end 60.081667 59.468333) (width 0.25) (layer "F.Cu") (net 23))
-  (segment (start 61.868333 59.468333) (end 62.65 60.25) (width 0.25) (layer "F.Cu") (net 23))
-  (segment (start 60.081667 59.468333) (end 59.675 59.875) (width 0.25) (layer "F.Cu") (net 23))
-  (segment (start 60.9625 59.468333) (end 61.868333 59.468333) (width 0.25) (layer "F.Cu") (net 23))
+  (segment (start 59 48.3) (end 59 54.1) (width 0.25) (layer "B.Cu") (net 22))
+  (segment (start 68.7 61.9) (end 70.4875 63.6875) (width 0.25) (layer "F.Cu") (net 23))
+  (segment (start 62.4 61.9) (end 68.7 61.9) (width 0.25) (layer "F.Cu") (net 23))
+  (segment (start 60.062 61.038) (end 60.9625 60.1375) (width 0.25) (layer "F.Cu") (net 23))
   (segment (start 35.5 64.9) (end 35.5 62.4) (width 0.25) (layer "F.Cu") (net 23))
-  (segment (start 70.4875 65.9125) (end 69 67.4) (width 0.25) (layer "F.Cu") (net 23))
+  (segment (start 60.9625 59.468333) (end 60.9625 60.4625) (width 0.25) (layer "F.Cu") (net 23))
   (segment (start 38.1 59.8) (end 53.312 59.8) (width 0.25) (layer "F.Cu") (net 23))
-  (segment (start 62.25 59.85) (end 62.136666 59.736666) (width 0.25) (layer "F.Cu") (net 23))
-  (segment (start 58.512 61.038) (end 54.55 61.038) (width 0.25) (layer "F.Cu") (net 23))
-  (segment (start 69 67.4) (end 64.5 67.4) (width 0.25) (layer "F.Cu") (net 23))
-  (segment (start 63 65.9) (end 63 60.6) (width 0.25) (layer "F.Cu") (net 23))
-  (segment (start 63 60.6) (end 62.65 60.25) (width 0.25) (layer "F.Cu") (net 23))
-  (segment (start 64.5 67.4) (end 63 65.9) (width 0.25) (layer "F.Cu") (net 23))
-  (segment (start 61.868333 59.468333) (end 62.25 59.85) (width 0.25) (layer "F.Cu") (net 23))
+  (segment (start 60.9625 60.1375) (end 60.9625 59.468333) (width 0.25) (layer "F.Cu") (net 23))
+  (segment (start 60.9625 60.4625) (end 62.4 61.9) (width 0.25) (layer "F.Cu") (net 23))
   (segment (start 35.5 62.4) (end 38.1 59.8) (width 0.25) (layer "F.Cu") (net 23))
+  (segment (start 54.55 61.038) (end 60.062 61.038) (width 0.25) (layer "F.Cu") (net 23))
   (segment (start 53.312 59.8) (end 54.55 61.038) (width 0.25) (layer "F.Cu") (net 23))
-  (segment (start 62.65 60.25) (end 62.25 59.85) (width 0.25) (layer "F.Cu") (net 23))
-  (segment (start 71 68.7) (end 72.2 67.5) (width 0.25) (layer "F.Cu") (net 24))
   (segment (start 41.85 61.038) (end 45.148667 64.336667) (width 0.25) (layer "F.Cu") (net 24))
   (segment (start 60.9625 64.336667) (end 45.148667 64.336667) (width 0.25) (layer "F.Cu") (net 24))
-  (segment (start 63.3 68.7) (end 71 68.7) (width 0.25) (layer "F.Cu") (net 24))
-  (segment (start 60.9625 64.336667) (end 60.9625 66.3625) (width 0.25) (layer "F.Cu") (net 24))
-  (segment (start 72.2 67.5) (end 72.2 60.7) (width 0.25) (layer "F.Cu") (net 24))
+  (segment (start 72 60.5) (end 71.7 60.2) (width 0.25) (layer "F.Cu") (net 24))
+  (segment (start 71.3 66.9) (end 72 66.2) (width 0.25) (layer "F.Cu") (net 24))
+  (segment (start 72 66.2) (end 72 60.5) (width 0.25) (layer "F.Cu") (net 24))
   (segment (start 70.968333 59.468333) (end 71.7 60.2) (width 0.25) (layer "F.Cu") (net 24))
-  (segment (start 72.2 60.7) (end 71.7 60.2) (width 0.25) (layer "F.Cu") (net 24))
   (segment (start 71.7 60.2) (end 71.236666 59.736666) (width 0.25) (layer "F.Cu") (net 24))
-  (segment (start 60.9625 66.3625) (end 63.3 68.7) (width 0.25) (layer "F.Cu") (net 24))
+  (segment (start 60.9625 66.2125) (end 61.65 66.9) (width 0.25) (layer "F.Cu") (net 24))
+  (segment (start 61.65 66.9) (end 71.3 66.9) (width 0.25) (layer "F.Cu") (net 24))
+  (segment (start 60.9625 64.336667) (end 60.9625 66.2125) (width 0.25) (layer "F.Cu") (net 24))
   (segment (start 25.975 64.9) (end 25.975 62.625) (width 0.25) (layer "F.Cu") (net 25))
   (segment (start 29.9 58.7) (end 53.332 58.7) (width 0.25) (layer "F.Cu") (net 25))
